File: takone.kicad_pcb (KiCad board)
At the start: 4 copper layers, 320 x 53 mm, 241 parts, among them J1 Conn_01x01, J10 Conn_01x03, J11 Conn_01x03, J12 Conn_01x04, J13 Conn_01x04, J14 Conn_01x04, J15 Conn_01x03, J16 Conn_01x03, J17 Conn_01x03, J18 Conn_01x08, J19 Conn_02x02_Counter_Clockwise, J2 Conn_01x01, J20 Conn_02x02_Counter_Clockwise, J21 Conn_02x02_Counter_Clockwise, J22 Conn_02x02_Counter_Clockwise, J23 Conn_02x02_Counter_Clockwise, J24 Conn_02x02_Counter_Clockwise, J25 Conn_02x02_Counter_Clockwise, J26 Conn_02x02_Counter_Clockwise, J3 Conn_01x03, J4 Conn_01x03, J5 Conn_01x03, J6 Conn_01x03, J7 Conn_01x03, J8 Conn_01x03, J9 Conn_01x03, Q1 SS8050, Q10 SS8050, Q11 SS8050, Q12 SS8050, Q13 SS8050, Q14 SS8050, Q15 SS8050, Q16 SS8050, Q17 SS8050, Q18 SS8050, Q19 PSMN028-100YS, Q2 SS8050, Q20 PSMN028-100YS, Q21 PSMN028-100YS, Q22 SS8050, Q23 SS8050, Q24 SS8050, Q25 SS8050, Q26 SS8050, Q27 SS8050, Q28 SS8050, Q29 PSMN028-100YS, Q3 SS8050, Q30 PSMN028-100YS, Q31 SS8050, Q32 SS8050, Q4 SS8050, Q5 SS8050, Q6 SS8050, Q7 PSMN028-100YS, Q8 PSMN028-100YS, Q9 PSMN028-100YS, U1 ADM3488ARZ, U10 Relay, U11 INA180, U12 Relay, U13 INA180, U14 INA180, U15 Relay, U16 Relay, U17 Relay, U18 Relay, U19 Relay, U2 ADM3488ARZ, U20 INA180, U21 Relay, U22 INA180, U23 INA180, U24 Relay, U25 Relay, U26 Relay, U27 Relay, U28 INA180, U29 INA180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

Commit message: correctif empreintes
Parts:
- removed ? (x2): MountingHole_3.2mm_M3, Mounting_Holes:MountingHole_3.2mm_M3
- R10, R11, R13, R15, R27, R30, R31, R32, R33, R34, R35, R37, R39, R51, R54, R55, R56, R57, R58, R60, R70, R71, R8, R9: value 3.9k -> 680R
- U1, U2, U3: value ADM3488ARZ -> R_8
- U5: value STM32G0_LQFP64_T1 -> LQFP-64
- moved R71 14.3 mm to (378.4, 137.5), turned to 90 degrees
- moved R54 13.4 mm to (322.4, 136.9), turned to 90 degrees
- moved Q23 10.2 mm to (320.6, 139.7), turned to 180 degrees
- moved Q32 10.0 mm to (375.6, 139.7), turned to 180 degrees
- moved G*** 5.47 mm to (188.3, 147.4)
- moved R27 4.97 mm to (113.5, 134.3), turned to 90 degrees
- moved D23 3.40 mm to (316.6, 139.3)
- moved D32 3.36 mm to (371.8, 139.4)
- moved R51 2.44 mm to (174.8, 138.8)
- moved Q22 2.34 mm to (171.7, 139.7), turned to 180 degrees
- moved D22 2.29 mm to (167.8, 139.5)
- moved D10 2.15 mm to (111.8, 139.2)
- moved R70 2.10 mm to (78.5, 166.9)
- moved R30 2.01 mm to (133.8, 167.2)
- moved Q10 1.80 mm to (115.7, 139.0), turned to 180 degrees
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Connections:
- J2 pad 1: (no net) -> GNDREF
- Q1 pad 1: GND -> Net-(Q1-Pad1)
- Q1 pad 2: Net-(Q1-Pad2) -> GND
- Q10 pad 1: GND -> Net-(Q10-Pad1)
- Q10 pad 2: Net-(Q10-Pad2) -> GND
- Q11 pad 1: GND -> Net-(Q11-Pad1)
- Q11 pad 2: Net-(Q11-Pad2) -> GND
- Q12 pad 1: GND -> Net-(Q12-Pad1)
- Q12 pad 2: Net-(Q12-Pad2) -> GND
- Q13 pad 1: GND -> Net-(Q13-Pad1)
- Q13 pad 2: Net-(Q13-Pad2) -> GND
- Q14 pad 1: GND -> Net-(Q14-Pad1)
- Q14 pad 2: Net-(Q14-Pad2) -> GND
- Q15 pad 1: GND -> Net-(Q15-Pad1)
- Q15 pad 2: Net-(Q15-Pad2) -> GND
- Q16 pad 1: GND -> Net-(Q16-Pad1)
- Q16 pad 2: Net-(Q16-Pad2) -> GND
- Q17 pad 1: GND -> Net-(Q17-Pad1)
- Q17 pad 2: Net-(Q17-Pad2) -> GND
- Q18 pad 1: GND -> Net-(Q18-Pad1)
- Q18 pad 2: Net-(Q18-Pad2) -> GND
- Q2 pad 1: GND -> Net-(Q2-Pad1)
- Q2 pad 2: Net-(Q2-Pad2) -> GND
- Q22 pad 1: GND -> Net-(Q22-Pad1)
- Q22 pad 2: Net-(Q22-Pad2) -> GND
- Q23 pad 1: GND -> Net-(Q23-Pad1)
- Q23 pad 2: Net-(Q23-Pad2) -> GND
- Q24 pad 1: GND -> Net-(Q24-Pad1)
- Q24 pad 2: Net-(Q24-Pad2) -> GND
- Q25 pad 1: GND -> Net-(Q25-Pad1)
- Q25 pad 2: Net-(Q25-Pad2) -> GND
- Q26 pad 1: GND -> Net-(Q26-Pad1)
- Q26 pad 2: Net-(Q26-Pad2) -> GND
- Q27 pad 1: GND -> Net-(Q27-Pad1)
- Q27 pad 2: Net-(Q27-Pad2) -> GND
- Q28 pad 1: GND -> Net-(Q28-Pad1)
- Q28 pad 2: Net-(Q28-Pad2) -> GND
- Q3 pad 1: GND -> Net-(Q3-Pad1)
- Q3 pad 2: Net-(Q3-Pad2) -> GND
- Q31 pad 1: GND -> Net-(Q31-Pad1)
- Q31 pad 2: Net-(Q31-Pad2) -> GND
- Q32 pad 1: GND -> Net-(Q32-Pad1)
- Q32 pad 2: Net-(Q32-Pad2) -> GND
- Q4 pad 1: GND -> Net-(Q4-Pad1)
- Q4 pad 2: Net-(Q4-Pad2) -> GND
- Q5 pad 1: GND -> Net-(Q5-Pad1)
- Q5 pad 2: Net-(Q5-Pad2) -> GND
- Q6 pad 1: GND -> Net-(Q6-Pad1)
- Q6 pad 2: Net-(Q6-Pad2) -> GND
- R10 pad 2: Net-(Q3-Pad2) -> Net-(Q3-Pad1)
- R11 pad 1: Net-(Q4-Pad2) -> Net-(Q4-Pad1)
- R13 pad 1: Net-(Q5-Pad2) -> Net-(Q5-Pad1)
- R15 pad 1: Net-(Q6-Pad2) -> Net-(Q6-Pad1)
- R27 pad 1: Net-(Q10-Pad2) -> Net-(Q10-Pad1)
- R30 pad 1: Net-(Q11-Pad2) -> Net-(Q11-Pad1)
- R31 pad 1: Net-(Q12-Pad2) -> Net-(Q12-Pad1)
- R32 pad 2: Net-(Q13-Pad2) -> Net-(Q13-Pad1)
- R33 pad 2: Net-(Q14-Pad2) -> Net-(Q14-Pad1)
- R34 pad 2: Net-(Q15-Pad2) -> Net-(Q15-Pad1)
- R35 pad 1: Net-(Q16-Pad2) -> Net-(Q16-Pad1)
- R37 pad 1: Net-(Q17-Pad2) -> Net-(Q17-Pad1)
- R39 pad 1: Net-(Q18-Pad2) -> Net-(Q18-Pad1)
- R51 pad 1: Net-(Q22-Pad2) -> Net-(Q22-Pad1)
- R54 pad 1: Net-(Q23-Pad2) -> Net-(Q23-Pad1)
- R55 pad 1: Net-(Q24-Pad2) -> Net-(Q24-Pad1)
- R56 pad 2: Net-(Q25-Pad2) -> Net-(Q25-Pad1)
- R57 pad 2: Net-(Q26-Pad2) -> Net-(Q26-Pad1)
- R58 pad 1: Net-(Q27-Pad2) -> Net-(Q27-Pad1)
- R60 pad 1: Net-(Q28-Pad2) -> Net-(Q28-Pad1)
- R70 pad 1: Net-(Q31-Pad2) -> Net-(Q31-Pad1)
- R71 pad 1: Net-(Q32-Pad2) -> Net-(Q32-Pad1)
- R8 pad 2: Net-(Q1-Pad2) -> Net-(Q1-Pad1)
- R9 pad 2: Net-(Q2-Pad2) -> Net-(Q2-Pad1)
- U5 pad 16: (no net) -> Net-(U5-Pad16)
- U5 pad 30: (no net) -> Net-(U5-Pad30)
- U5 pad 31: (no net) -> Net-(U5-Pad31)
- U5 pad 32: (no net) -> Net-(U5-Pad32)
- U5 pad 40: (no net) -> Net-(U5-Pad40)
- U5 pad 41: (no net) -> Net-(U5-Pad41)
Routing:
- net +12V: track 189.3 -> 421.3 mm, vias 9 -> 22
- net GND: track 205.9 -> 107.6 mm, vias 36 -> 28
- net (no net): track 28.8 -> 0.00 mm
- net GNDREF: track 0.00 -> 28.8 mm
- net GNDA: track 94.2 -> 112.4 mm
- net RELAY10: track 126.0 -> 143.6 mm
- net RELAY12: track 185.0 -> 199.2 mm
- net Net-(D24-Pad1): track 9.66 -> 21.8 mm
- net MOS7: track 102.9 -> 95.9 mm
- net RELAY6: track 162.0 -> 168.8 mm
- net Net-(Q10-Pad1): track 0.00 -> 6.32 mm
- net RELAY8: track 110.9 -> 117.3 mm
- net Net-(Q14-Pad2): track 5.84 -> 0.00 mm
- net Net-(Q15-Pad2): track 5.26 -> 0.00 mm
- net Net-(Q2-Pad2): track 5.08 -> 0.00 mm
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